File: tp4056-multicell-charger.kicad_sch (KiCad schematic)
At the start: 21 parts, among them J1 USB_C_Receptacle_PowerOnly_6P, J2 Conn_01x03, J3 Conn_01x04, J4 Conn_01x03, J5 Conn_01x04, U1 TP4056, U2 TP4056, U3 TP4056

Commit message: fixed title *.pdfを除外
Other:
- title: tp4056-multicell-charger -> TP4056 Multicell Charger
Changed lines of the file:
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@@
 	(paper "A4")
 	(title_block
-		(title "tp4056-multicell-charger")
-		(date "2026-10-07")
+		(title "TP4056 Multicell Charger")
+		(date "2026-10-15")
 		(rev "1.0")
 	)

Commit message: footprint edit
Parts:
- U1, U2, U3: footprint Charger_Module:TP4056_Module -> Charger_Module:TP4056_Module_SMD
Changed lines of the file:
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@@
 			)
 		)
-		(property "Footprint" "Charger_Module:TP4056_Module"
+		(property "Footprint" "Charger_Module:TP4056_Module_SMD"
 			(at 144.78 83.82 0)
 			(hide yes)
@@
 			)
 		)
-		(property "Footprint" "Charger_Module:TP4056_Module"
+		(property "Footprint" "Charger_Module:TP4056_Module_SMD"
 			(at 144.78 60.96 0)
 			(hide yes)
@@
 			)
 		)
-		(property "Footprint" "Charger_Module:TP4056_Module"
+		(property "Footprint" "Charger_Module:TP4056_Module_SMD"
 			(at 144.78 35.56 0)
 			(hide yes)
