File: tp4056-multicell-charger.kicad_pcb (KiCad board)
At the start: 2 copper layers, 60 x 40 mm, 11 parts, among them J1 USB_C_Receptacle_PowerOnly_6P, J2 Conn_01x03, J3 Conn_01x04

Commit message: footprint edit
Parts:
- added U1: TP4056, Charger_Module:TP4056_Module_SMD, F.Cu at (101.8, 90.5)
- added U2: TP4056, Charger_Module:TP4056_Module_SMD, F.Cu at (101.8, 109.5)
- added U3: TP4056, Charger_Module:TP4056_Module_SMD, B.Cu at (101.8, 109.5)
Routing:
- net Cell2+: track 0.00 -> 37.4 mm
- net Cell1+: track 0.00 -> 31.3 mm, vias 0 -> 9
- net Cell1-: track 0.00 -> 24.8 mm
- net +5V: track 27.1 -> 42.5 mm
- net GND: track 49.5 -> 64.8 mm, vias 0 -> 69
- net Net-(PS1-0V): track 3.09 -> 14.5 mm
- net Cell3+: track 0.00 -> 11.3 mm, vias 0 -> 1
- net Net-(PS2-+Vo): track 3.96 -> 14.9 mm
- net Net-(PS2-0V): track 3.09 -> 12.7 mm
- net Net-(PS1-+Vo): track 3.96 -> 11.5 mm
- net Net-(J1-CC2): track 8.50 -> 9.01 mm

Commit message: add REVISION value
Other:
- board text added: "Rev ${REVISION}"
Changed lines of the file:
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@@
 		)
 	)
+	(property "REVISION" "v1.0.0")
 	(footprint "Connector_JST:JST_XH_S4B-XH-A_1x04_P2.50mm_Horizontal"
 		(layer "F.Cu")
@@
 		)
 	)
+	(gr_text "Rev ${REVISION}"
+		(at 117 119 0)
+		(layer "F.SilkS")
+		(effects
+			(font
+				(size 1 1)
+				(bold yes)
+			)
+			(justify left bottom)
+		)
+	)

Commit message: add via to Cell3+
Routing:
- net Cell3+: vias 1 -> 2
Changed lines of the file:
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@@
+		(net "Cell3+")
+	)
+	(via
+		(at 112.9 87.75)
+		(size 0.6)
+		(drill 0.3)
+		(layers "F.Cu" "B.Cu")
 		(net "Cell3+")
 	)
